File: front-panel-usb.kicad_sch (KiCad schematic)
At the start: 87 parts, among them J2 USB-C_Kycon_KUSBX-SL2-CS1N24-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, J3 USB-C_Kycon_KUSBX-SL2-CS1N24-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, J4 USB-C_Kycon_KUSBX-SL2-CS1N24-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, Q1 BSS84AKW, U10 TPD4E05U06QDQARQ1, U21 TUSB321RWBR, U22 TUSB321RWBR, U4 TPD4E05U06QDQARQ1, U5 FT4232H_VQFN, U6 NCP718BSN330T1G, U7 AP22615A_TSOT26, U8 AP22615A_TSOT26, U9 TPD4E05U06QDQARQ1, Y1 Resonator_12MHz_ABM8G

Commit message: [#83336] Improved USB circuitry
Parts:
- removed C20: C_1u_25V_0402, antmicro-footprints:C_0402_1005Metric, symbol antmicroCapacitors0402:C_1u_25V_0402
- removed C22, C62, C63: C_100n_0402, antmicro-footprints:C_0402_1005Metric, symbol antmicroCapacitors0402:C_100n_0402
- removed D3, D4: DF2S30FS_SOD, antmicro-footprints:SOD-923, symbol antmicroTVSDiodes:DF2S30FS_SOD
- removed Q1: BSS84AKW, antmicro-footprints:SOT-323, symbol antmicroTransistorsFETsMOSFETsSingle:BSS84AKW
- removed R12, R13: R_5k11_0402, antmicro-footprints:R_0402_1005Metric, symbol antmicroResistors0402:R_5k11_0402
- removed R22, R23, R24, R25, R26: R_0R_0402, antmicro-footprints:R_0402_1005Metric, symbol antmicroResistors0402:R_0R_0402
- removed R28, R68: R_887k_0402, antmicro-footprints:R_0402_1005Metric, symbol Resistors0402:R_887k_0402
- removed R30: R_10k_0402, antmicro-footprints:R_0402_1005Metric, symbol antmicroResistors0402:R_10k_0402
- removed R31, R35: R_8k2_0402, antmicro-footprints:R_0402_1005Metric, symbol Resistors0402:R_8k2_0402
- removed R32, R34: R_4k7_0402, antmicro-footprints:R_0402_1005Metric, symbol Resistors0402:R_4k7_0402
- removed R33, R36: R_10k_0402, antmicro-footprints:R_0402_1005Metric, symbol Resistors0402:R_10k_0402
- removed R38: R_330R_0402, antmicro-footprints:R_0402_1005Metric, symbol antmicroResistors0402:R_330R_0402
- removed U10: TPD4E05U06QDQARQ1, antmicro-footprints:USON-10_2.5x1mm_P0.5mm, symbol antmicroTVSDiodes:TPD4E05U06QDQARQ1
- removed U21, U22: TUSB321RWBR, antmicro-footprints:Texas_X2QFN-12_1.6x1.6mm_P0.4mm, symbol InterfaceControllers:TUSB321RWBR
- added C154, C20: C_100n_0402, antmicro-footprints:C_0402_1005Metric, symbol antmicroCapacitors0402:C_100n_0402
- added C22: C_1u_25V_0402, antmicro-footprints:C_0402_1005Metric, symbol antmicroCapacitors0402:C_1u_25V_0402
- added D10, D3: PESD5V0X1UB, antmicro-footprints:SOD-523, symbol antmicroTVSDiodes:PESD5V0X1UB
- added R12, R210: R_5k1_0201, antmicro-footprints:R_0201, symbol antmicroResistorsmisc:R_5k1_0201
- added R13, R211, R22, R23, R24, R25, R26, R28, R31, R35, R38, R68: R_10k_0402, antmicro-footprints:R_0402_1005Metric, symbol antmicroResistors0402:R_10k_0402
- added R212, R32: R_3k16_0402, antmicro-footprints:R_0402_1005Metric, symbol antmicroResistors0402:R_3k16_0402
- added R213: R_330R_0402, antmicro-footprints:R_0402_1005Metric, symbol antmicroResistors0402:R_330R_0402
- added R30, R33, R34, R36: R_910k_0402, antmicro-footprints:R_0402_1005Metric, symbol antmicroResistors0402:R_910k_0402
- added TP3, TP5, TP9: TP_0.75mm_SMD, antmicro-footprints:TP_SMD_0.75mm, symbol antmicroTestPoints:TP_0.75mm_SMD
- added U10, U21: FUSB303B, antmicro-footprints:Texas_X2QFN-12_1.6x1.6mm_P0.4mm, symbol antmicroInterfaceControllers:FUSB303B
- added U22: TPD4E05U06QDQARQ1, antmicro-footprints:USON-10_2.5x1mm_P0.5mm, symbol antmicroTVSDiodes:TPD4E05U06QDQARQ1
- added U33: 74LVC06ABQ, antmicro-footprints:DHVQFN-14-1EP_2.5x3mm, symbol antmicroLogicBuffersDriversReceiversTransceivers:74LVC06ABQ
- R27: now not fitted
Connections:
- net +5V: now also C25.2, R29.1, C20.2, R13.2, R23.2, R28.1, R31.1, R33.2, R35.1, R36.2, R38.2, R68.2, U10.12 (V_{DD}), U21.12 (V_{DD}); no longer C25.1, C61.1, R27.2
- net FTDI_3V3: now also D2.2 (A)
- net GND: now also C25.1, R27.2, C154.1, C20.1, C22.2, D10.2 (A), D3.2 (A), R12.2, R210.2, R211.2, R212.1, R213.2, R22.2, R24.2, R25.2, R26.2, R30.2, R32.1, R34.2, U10.10 (GND), U21.10 (GND), U22.3, U22.8, U33.11 (5A), U33.13 (6A), U33.15 (GND), U33.7 (GND), U33.9 (4A); no longer C25.2, R29.1, R53.1, R54.1, R55.1
- net LED0: now also U33.1 (1A)
- net LED1: now also U33.3 (2A)
- net LED2: now also U33.5 (3A)
- net USB0_CC1: now also U21.1 (CC1)
- net USB0_CC2: now also U21.2 (CC2)
- net USB0_VBUS: now also D10.1 (C), U21.4 (VBUS_{DET})
- net USB1.D+: now also U22.2, U22.9
- net USB1.D-: now also U22.4, U22.7
- net USB1_CC1: now also U10.1 (CC1), U22.1, U22.10
- net USB1_CC2: now also U10.2 (CC2), U22.5, U22.6
- net USB1_VBUS: now also C24.1, C22.1, D3.1 (C), U10.4 (VBUS_{DET})
- net USB2_CC1: now also R210.1
- net USB2_CC2: now also R12.1
- net at D7.1 (C): now also U33.4 (2Y); no longer R54.2
- net at D7.2 (A): now also R54.1
- net ID2: now reaches U8.4 (EN)
- net ID2: now also R68.1, U10.9 (ID)
- net at D8.1 (C): now also U33.6 (3Y); no longer R55.2
- net at U8.5 (ISET): now also R212.2
- net ID1: now reaches U7.4 (EN)
- net ID1: now also R13.1, U21.9 (ID); no longer R29.2
- net at U7.5 (ISET): now also R32.2
- net at J4.SH: now also C61.1, R213.1; no longer C24.1
- net at D6.1 (C): now also U33.2 (1Y); no longer R53.2
- net at D6.2 (A): now also R53.1
- net at D8.2 (A): now also R55.1
- removed net USBC0_FLG: R27.1, TP4.1, U7.3 (FLG)
- net USBC1_FLG renamed FLG2
- net FLG2: now also R38.1
- new net: TP9.1, U10.5 (ADDR/ORIENT)
- new net: TP4.1, U10.6 (~{INT}/OUT3)
- new net: R211.1, U10.11 (~{EN})
- new net: TP3.1, U21.5 (ADDR/ORIENT)
- new net: TP5.1, U21.6 (~{INT}/OUT3)
- new net: R22.1, U21.11 (~{EN})
- new net +1V8: C154.2, U33.14 (V_{CC})
- new net +3V3: R53.2, R54.2, R55.2
- new net FLG1: R23.1, U7.3 (FLG)
- new net PORT0: R33.1, R34.1, U21.3 (PORT/~{DEBUG})
- new net PORT2: R30.1, R36.1, U10.3 (PORT/~{DEBUG})
- new net SCL0: R27.1, R29.2, U21.8 (SCL/OUT2)
- new net SCL2: R26.1, R35.2, U10.8 (SCL/OUT2)
- new net SDA0: R25.1, R28.2, U21.7 (SDA/OUT1)
- new net SDA1: R24.1, R31.2, U10.7 (SDA/OUT1)
- no-connect marks 67 -> 61
Other:
- note added: "Ilimit set to 2A"
- note added: "SINK ONLY Can be reconfigured as UFP or DRP with R33 and R34"
- note added: "SOURCE ONLY Can be reconfigured as UFP or DRP with R33 and R34"
- note removed: "Advertise as 500mA source"
- note removed: "DFP"
- note removed: "Ilimit set to 0.7A"
- note removed: "USB-C 2"
- moved on the sheet: C17, C19, C21, D2, D6, D7, D8, H2, R21, R53, R54, R55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

Commit message: [#83336] Small front panel interface fixes
Parts:
- removed C19, C22: C_1u_25V_0402, antmicro-footprints:C_0402_1005Metric, symbol antmicroCapacitors0402:C_1u_25V_0402
- removed J2, J3, J4: USB-C_Kycon_KUSBX-SL2-CS1N24-B-TR, antmicro-footprints:USB-C_Receptacle_Kycon_KUSBX-SL2-CS1N24-B-TR, symbol antmicroUSBConnectors:USB-C_Kycon_KUSBX-SL2-CS1N24-B-TR
- removed U7, U8: AP22615A_TSOT26, antmicro-footprints:TSOT23-6, symbol antmicroPMICPowerDistributionSwitchesLoadDrivers:AP22615A_TSOT26
- added C19, C62: C_4u7_0402, antmicro-footprints:C_0402_1005Metric, symbol antmicroCapacitors0402:C_4u7_0402
- added D11, D5: LED_G_0402_VLMTG1500-GS08, antmicro-footprints:LED_0402_1005Metric_G, symbol antmicroLEDIndicationDiscrete:LED_G_0402_VLMTG1500-GS08
- added J2, J3, J6: USB-C_GCT_USB4105-GF-A, antmicro-footprints:USB-C_Receptacle_GCT_USB4105-GF-A, symbol antmicroUSBConnectors:USB-C_GCT_USB4105-GF-A
- added J4: Tag-Connect_TC2050-IDC-NL_2x5_P1.27mm, antmicro-footprints:Tag-Connect_TC2050-IDC-NL_2x5_P1.27mm, symbol antmicroTestPoints:Tag-Connect_TC2050-IDC-NL_2x5_P1.27mm
- added Q1: PJE138K, antmicro-footprints:SOT-523, symbol antmicroTransistorsFETsMOSFETsSingle:PJE138K
- added R214, R215: R_330R_0402, antmicro-footprints:R_0402_1005Metric, symbol antmicroResistors0402:R_330R_0402
- added R216: R_100k_0402, antmicro-footprints:R_0402_1005Metric, symbol antmicroResistors0402:R_100k_0402
- added R217, R218, R219, R220, R221, R222: R_0R_0402, antmicro-footprints:R_0402_1005Metric, symbol antmicroResistors0402:R_0R_0402
- added TP10: TP_0.75mm_SMD, antmicro-footprints:TP_SMD_0.75mm, symbol antmicroTestPoints:TP_0.75mm_SMD
- added U7, U8: AP22615B_TSOT26, antmicro-footprints:TSOT23-6, symbol antmicroPMICPowerDistributionSwitchesLoadDrivers:AP22615B_TSOT26
- R38: now not fitted
Connections:
- net FLG2 is gone; now on net FLG1: R38.1
- net ID2 is gone; now on net ID1: R68.1, U10.9 (ID)
- net +5V: now also U7.6 (IN), U8.6 (IN)
- net FLG1: now also R217.2, U8.3 (FLG); no longer R23.1
- net GND: now also C19.1, C62.1, D11.1 (C), D5.1 (C), J2.A1 (GND), J2.A12 (GND), J2.B1 (GND), J2.B12 (GND), J3.A1 (GND), J3.A12 (GND), J3.B1 (GND), J3.B12 (GND), J4.3, J4.5, J4.9, J6.A1 (GND), J6.A12 (GND), J6.B1 (GND), J6.B12 (GND), Q1.2 (S), R216.1, U7.2 (GND), U8.2 (GND); no longer R211.2
- net ID1: now also U8.4 (~{EN}); no longer R13.1, U21.9 (ID)
- net JTAG.TCK: now also J4.4, R218.2; no longer U5.12 (ADBUS0)
- net JTAG.TDI: now also J4.8, R219.2; no longer U5.13 (ADBUS1)
- net JTAG.TDO: now also J4.6, R220.2; no longer U5.14 (ADBUS2)
- net JTAG.TMS: now also J4.2, R221.2; no longer U5.15 (ADBUS3)
- net USB0.D+: now also J6.A6 (D_{A}+), J6.B6 (D_{B}+)
- net USB0.D-: now also J6.A7 (D_{A}-), J6.B7 (D_{B}-)
- net USB0_CC1: now also J6.A5 (CC_{1})
- net USB0_CC2: now also J6.B5 (CC_{2})
- net USB0_VBUS: now also C62.2, J6.A4 (VBUS), J6.A9 (VBUS), J6.B4 (VBUS), J6.B9 (VBUS), R215.2, U7.1 (OUT)
- net USB1.D+: now also J3.A6 (D_{A}+), J3.B6 (D_{B}+)
- net USB1.D-: now also J3.A7 (D_{A}-), J3.B7 (D_{B}-)
- net USB1_CC1: now also J3.A5 (CC_{1})
- net USB1_CC2: now also J3.B5 (CC_{2})
- net USB1_VBUS: now also C19.2, J3.A4 (VBUS), J3.A9 (VBUS), J3.B4 (VBUS), J3.B9 (VBUS), R214.2, U8.1 (OUT)
- net USB2_CC1: now also J2.A5 (CC_{1})
- net USB2_CC2: now also J2.B5 (CC_{2})
- net USB2_D+: now also J2.A6 (D_{A}+), J2.B6 (D_{B}+)
- net USB2_D-: now also J2.A7 (D_{A}-), J2.B7 (D_{B}-)
- net USB2_VBUS: now also J2.A4 (VBUS), J2.A9 (VBUS), J2.B4 (VBUS), J2.B9 (VBUS)
- net at R212.2: now also U8.5 (ISET)
- net at C61.1, R213.1: now also J3.SH
- net at C23.1, R37.1: now also J6.SH
- net at R32.2: now also U7.5 (ISET)
- net at C11.1, R11.1: now also J2.SH
- new net: D11.2 (A), R215.1
- new net: R219.1, U5.13 (ADBUS1)
- new net: J4.10, TP10.1
- new net: R221.1, U5.15 (ADBUS3)
- new net: Q1.3 (D), R211.2
- new net: R218.1, U5.12 (ADBUS0)
- new net: R220.1, U5.14 (ADBUS2)
- new net: J4.1, R222.2
- new net: D5.2 (A), R214.1
- new net +3V3_AON: R222.1
- new net FLG0: R23.1, U7.3 (FLG)
- new net ID0: R13.1, U21.9 (ID), U7.4 (~{EN})
- new net USBC1_5V_PEN: Q1.1 (G), R216.2
- new net USBC1_FLG: R217.1
- no-connect marks 61 -> 37
Other:
- note added: "MCU LEDs"
- note removed: "LEDs"
- moved on the sheet: C11, C23, C61, R11, R12, R17, R18, R19, R20, R210, R213, R37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
