File: front-panel-ethernet.kicad_sch (KiCad schematic)
At the start: 7 parts, among them J9 Bus_RJ45_7498111120R

Commit message: [#83609] Reannotate board
Parts:
- renumbered C22 to C81, J9 to J8, R41 to R191, R39 to R192, R40 to R193
Changed lines of the file:
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@@
 		(dnp no)
 		(fields_autoplaced yes)
-		(property "Reference" "J9"
+		(property "Reference" "J8"
 			(at 226.06 114.3 0)
 			(effects
@@
 			(project ""
 				(path "/5f636c45-3c15-4731-8931-4625e0dab7e4/9da0fa42-de01-45ef-a25f-792bb7803b7a"
-					(reference "J9")
+					(reference "J8")
 					(unit 1)
 				)
@@
 		(on_board yes)
 		(dnp no)
-		(property "Reference" "#PWR0203"
+		(property "Reference" "#PWR0175"
 			(at 233.68 162.56 0)
 			(effects
@@
 			(project "bmc-reference-carrier-board"
 				(path "/5f636c45-3c15-4731-8931-4625e0dab7e4/9da0fa42-de01-45ef-a25f-792bb7803b7a"
-					(reference "#PWR0203")
+					(reference "#PWR0175")
 					(unit 1)
 				)
@@
 		(on_board yes)
 		(dnp no)
-		(property "Reference" "#PWR051"
+		(property "Reference" "#PWR0172"
 			(at 182.88 162.56 0)
 			(effects
@@
 			(project "bmc-reference-carrier-board"
 				(path "/5f636c45-3c15-4731-8931-4625e0dab7e4/9da0fa42-de01-45ef-a25f-792bb7803b7a"
-					(reference "#PWR051")
+					(reference "#PWR0172")
 					(unit 1)
 				)
@@
 		(dnp no)
 		(fields_autoplaced yes)
-		(property "Reference" "R41"
+		(property "Reference" "R191"
 			(at 207.01 154.94 90)
 			(effects
@@
 			(project "bmc-reference-carrier-board"
 				(path "/5f636c45-3c15-4731-8931-4625e0dab7e4/9da0fa42-de01-45ef-a25f-792bb7803b7a"
-					(reference "R41")
+					(reference "R191")
 					(unit 1)
 				)
@@
 		(on_board yes)
 		(dnp no)
-		(property "Reference" "R39"
+		(property "Reference" "R192"
 			(at 243.84 143.51 90)
 			(effects
@@
 			(project ""
 				(path "/5f636c45-3c15-4731-8931-4625e0dab7e4/9da0fa42-de01-45ef-a25f-792bb7803b7a"
-					(reference "R39")
+					(reference "R192")
 					(unit 1)
 				)
@@
 		(on_board yes)
 		(dnp no)
-		(property "Reference" "#PWR052"
+		(property "Reference" "#PWR0173"
 			(at 196.85 166.37 0)
 			(effects
@@
 			(project "bmc-reference-carrier-board"
 				(path "/5f636c45-3c15-4731-8931-4625e0dab7e4/9da0fa42-de01-45ef-a25f-792bb7803b7a"
-					(reference "#PWR052")
+					(reference "#PWR0173")
 					(unit 1)
 				)
@@
 		(on_board yes)
 		(dnp no)
-		(property "Reference" "#PWR0204"
+		(property "Reference" "#PWR0176"
 			(at 260.35 111.76 0)
 			(effects
@@
 			(project "bmc-reference-carrier-board"
 				(path "/5f636c45-3c15-4731-8931-4625e0dab7e4/9da0fa42-de01-45ef-a25f-792bb7803b7a"
-					(reference "#PWR0204")
+					(reference "#PWR0176")
 					(unit 1)
 				)
@@
 		(on_board yes)
 		(dnp no)
-		(property "Reference" "C22"
+		(property "Reference" "C81"
 			(at 198.628 154.432 90)
 			(effects
@@
 			(project "bmc-reference-carrier-board"
 				(path "/5f636c45-3c15-4731-8931-4625e0dab7e4/9da0fa42-de01-45ef-a25f-792bb7803b7a"
-					(reference "C22")
+					(reference "C81")
 					(unit 1)
 				)
@@
 		(on_board yes)
 		(dnp no)
-		(property "Reference" "R40"
+		(property "Reference" "R193"
 			(at 246.888 115.57 90)
 			(effects
@@
 			(project "bmc-reference-carrier-board"
 				(path "/5f636c45-3c15-4731-8931-4625e0dab7e4/9da0fa42-de01-45ef-a25f-792bb7803b7a"
-					(reference "R40")
+					(reference "R193")
 					(unit 1)
 				)
@@
 		(on_board yes)
 		(dnp no)
-		(property "Reference" "#PWR053"
+		(property "Reference" "#PWR0174"
 			(at 204.47 166.37 0)
 			(effects
@@
 			(project "bmc-reference-carrier-board"
 				(path "/5f636c45-3c15-4731-8931-4625e0dab7e4/9da0fa42-de01-45ef-a25f-792bb7803b7a"
-					(reference "#PWR053")
+					(reference "#PWR0174")
 					(unit 1)
 				)
