File: front-panel-video.kicad_sch (KiCad schematic)
At the start: 23 parts, among them J9 DisplayPort-Mini_Pulse_E9320-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, U21 TPD4E05U06QDQARQ1, U22 TPD4E05U06QDQARQ1, U23 TPD4E05U06QDQARQ1

Commit message: [#83736] WIP: Clear ERC
Parts:
- J9: Manufacturer Pulse Electronics -> Pulse Electronics
Changed lines of the file:
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@@
 	)
 	(junction
+		(at 175.26 151.13)
+		(diameter 0)
+		(color 0 0 0 0)
+	)
+	(junction
 		(at 191.77 140.97)
 		(diameter 0)
@@
 	(wire
 		(pts
+			(xy 175.26 149.86) (xy 175.26 151.13)
+		)
+		(stroke
+			(width 0)
+			(type default)
+		)
+	)
+	(wire
+		(pts
 			(xy 269.24 147.32) (xy 261.62 147.32)
 		)
@@
 	(wire
 		(pts
-			(xy 167.64 151.13) (xy 177.8 151.13)
+			(xy 167.64 151.13) (xy 175.26 151.13)
 		)
 		(stroke
@@
 	(wire
 		(pts
+			(xy 175.26 151.13) (xy 177.8 151.13)
+		)
+		(stroke
+			(width 0)
+			(type default)
+		)
+	)
+	(wire
+		(pts
 			(xy 152.4 133.35) (xy 204.47 133.35)
 		)
@@
 	)
 	(symbol
+		(lib_name "DisplayPort-Mini_PulseElectronics_E9320-001-01_1")
+		(lib_id "antmicroVideoConnectors:DisplayPort-Mini_PulseElectronics_E9320-001-01")
+		(at 204.47 107.95 0)
+		(unit 1)
+		(exclude_from_sim no)
+		(in_bom yes)
+		(on_board yes)
+		(dnp no)
+		(fields_autoplaced yes)
+		(property "Reference" "J9"
+			(at 217.2335 100.33 0)
+			(effects
+				(font
+					(size 1.27 1.27)
+					(thickness 0.15)
+				)
+			)
+		)
+		(property "Value" "DisplayPort-Mini_Pulse_E9320-001-01"
+			(at 250.19 107.95 0)
+			(effects
+				(font
+					(size 1.27 1.27)
+					(thickness 0.15)
+				)
+				(justify left bottom)
+				(hide yes)
+			)
+		)
+		(property "Footprint" "antmicro-footprints:DisplayPort-Mini_Receptacle_Pulse_E9320-001-01"
+			(at 250.19 110.49 0)
+			(effects
+				(font
+					(size 1.27 1.27)
+					(thickness 0.15)
+				)
+				(justify left bottom)
+				(hide yes)
+			)
+		)
+		(property "Datasheet" "https://mm.digikey.com/Volume0/opasdata/d220001/medias/docus/6167/E9320-001-0x.pdf"
+			(at 250.19 113.03 0)
+			(effects
+				(font
+					(size 1.27 1.27)
+					(thickness 0.15)
+				)
+				(justify left bottom)
+				(hide yes)
+			)
+		)
+		(property "Description" "DisplayPort, Mini Receptacle Connector 20 Position THT/SMD, Right Angle"
+			(at 250.19 125.73 0)
+			(effects
+				(font
+					(size 1.27 1.27)
+				)
+				(justify left bottom)
+				(hide yes)
+			)
+		)
+		(property "MPN" "E9320-001-01"
+			(at 217.2335 102.87 0)
+			(effects
+				(font
+					(size 1.27 1.27)
+					(thickness 0.15)
+				)
+			)
+		)
+		(property "Manufacturer" "Pulse Electronics"
+			(at 250.19 118.11 0)
+			(effects
+				(font
+					(size 1.27 1.27)
+					(thickness 0.15)
+				)
+				(justify left bottom)
+				(hide yes)
+			)
+		)
+		(property "Author" "Antmicro"
+			(at 250.19 120.65 0)
+			(effects
+				(font
+					(size 1.27 1.27)
+					(thickness 0.15)
+				)
+				(justify left bottom)
+				(hide yes)
+			)
+		)
+		(property "License" "Apache-2.0"
+			(at 250.19 123.19 0)
+			(effects
+				(font
+					(size 1.27 1.27)
+					(thickness 0.15)
+				)
+				(justify left bottom)
+				(hide yes)
+			)
+		)
+		(pin "20"
+		)
+		(pin "16"
+		)
+		(pin "4"
+		)
+		(pin "1"
+		)
+		(pin "12"
+		)
+		(pin "10"
+		)
+		(pin "13"
+		)
+		(pin "2"
+		)
+		(pin "6"
+		)
+		(pin "8"
+		)
+		(pin "14"
+		)
+		(pin "5"
+		)
+		(pin "11"
+		)
+		(pin "7"
+		)
+		(pin "SH"
+		)
+		(pin "19"
+		)
+		(pin "9"
+		)
+		(pin "3"
+		)
+		(pin "15"
+		)
+		(pin "18"
+		)
+		(pin "17"
+		)
+		(instances
+			(project "bmc-reference-carrier-board"
+				(path "/5f636c45-3c15-4731-8931-4625e0dab7e4/32de8c9e-be2b-4d78-9d5d-f4e694f2d2e7"
+					(reference "J9")
+					(unit 1)
+				)
+			)
+		)
+	)
+	(symbol
 		(lib_id "antmicroCapacitors0402:C_100n_0402")
 		(at 144.78 138.43 180)
@@
 	)
 	(symbol
+		(lib_id "antmicropower:PWR_FLAG")
+		(at 175.26 149.86 0)
+		(unit 1)
+		(exclude_from_sim no)
+		(in_bom yes)
+		(on_board yes)
+		(dnp no)
+		(property "Reference" "#FLG01"
+			(at 175.26 147.955 0)
+			(effects
+				(font
+					(size 1.27 1.27)
+				)
+				(hide yes)
+			)
+		)
+		(property "Value" "PWR_FLAG"
+			(at 181.356 148.082 0)
+			(effects
+				(font
+					(size 1.27 1.27)
+				)
+			)
+		)
+		(property "Footprint" ""
+			(at 175.26 149.86 0)
+			(effects
+				(font
+					(size 1.27 1.27)
+				)
+				(hide yes)
+			)
+		)
+		(property "Datasheet" ""
+			(at 175.26 149.86 0)
+			(effects
+				(font
+					(size 1.27 1.27)
+				)
+				(hide yes)
+			)
+		)
+		(property "Description" ""
+			(at 175.26 149.86 0)
+			(effects
+				(font
+					(size 1.27 1.27)
+				)
+				(hide yes)
+			)
+		)
+		(pin "1"
+		)
+		(instances
+			(project ""
+				(path "/5f636c45-3c15-4731-8931-4625e0dab7e4/32de8c9e-be2b-4d78-9d5d-f4e694f2d2e7"
+					(reference "#FLG01")
+					(unit 1)
+				)
+			)
+		)
+	)
+	(symbol
 		(lib_id "antmicroCapacitors0402:C_100n_0402")
 		(at 152.4 133.35 180)
@@
 					(unit 1)
 				)
-			)
-		)
-	)
-	(symbol
-		(lib_id "antmicroVideoConnectors:DisplayPort-Mini_PulseElectronics_E9320-001-01")
-		(at 204.47 107.95 0)
-		(unit 1)
-		(exclude_from_sim no)
-		(in_bom yes)
-		(on_board yes)
-		(dnp no)
-		(fields_autoplaced yes)
-		(property "Reference" "J9"
-			(at 217.2335 100.33 0)
-			(effects
-				(font
-					(size 1.27 1.27)
-					(thickness 0.15)
-				)
-			)
-		)
-		(property "Value" "DisplayPort-Mini_Pulse_E9320-001-01"
-			(at 250.19 107.95 0)
-			(effects
-				(font
-					(size 1.27 1.27)
-					(thickness 0.15)
-				)
-				(justify left bottom)
-				(hide yes)
-			)
-		)
-		(property "Footprint" "antmicro-footprints:DisplayPort-Mini_Receptacle_Pulse_E9320-001-01"
-			(at 250.19 110.49 0)
-			(effects
-				(font
-					(size 1.27 1.27)
-					(thickness 0.15)
-				)
-				(justify left bottom)
-				(hide yes)
-			)
-		)
-		(property "Datasheet" "https://mm.digikey.com/Volume0/opasdata/d220001/medias/docus/6167/E9320-001-0x.pdf"
-			(at 250.19 113.03 0)
-			(effects
-				(font
-					(size 1.27 1.27)
-					(thickness 0.15)
-				)
-				(justify left bottom)
-				(hide yes)
-			)
-		)
-		(property "Description" "DisplayPort, Mini Receptacle Connector 20 Position THT/SMD, Right Angle"
-			(at 204.47 107.95 0)
-			(effects
-				(font
-					(size 1.27 1.27)
-				)
-				(hide yes)
-			)
-		)
-		(property "MPN" "E9320-001-01"
-			(at 217.2335 102.87 0)
-			(effects
-				(font
-					(size 1.27 1.27)
-					(thickness 0.15)
-				)
-			)
-		)
-		(property "Manufacturer" " Pulse Electronics"
-			(at 250.19 118.11 0)
-			(effects
-				(font
-					(size 1.27 1.27)
-					(thickness 0.15)
-				)
-				(justify left bottom)
-				(hide yes)
-			)
-		)
-		(property "Author" "Antmicro"
-			(at 250.19 120.65 0)
-			(effects
-				(font
-					(size 1.27 1.27)
-					(thickness 0.15)
-				)
-				(justify left bottom)
-				(hide yes)
-			)
-		)
-		(property "License" "Apache-2.0"
-			(at 250.19 123.19 0)
-			(effects
-				(font
-					(size 1.27 1.27)
-					(thickness 0.15)
-				)
-				(justify left bottom)
-				(hide yes)
-			)
-		)
-		(pin "16"
-		)
-		(pin "11"
-		)
-		(pin "14"
-		)
-		(pin "17"
-		)
-		(pin "6"
-		)
-		(pin "SH"
-		)
-		(pin "5"
-		)
-		(pin "4"
-		)
-		(pin "12"
-		)
-		(pin "10"
-		)
-		(pin "13"
-		)
-		(pin "20"
-		)
-		(pin "1"
-		)
-		(pin "15"
-		)
-		(pin "18"
-		)
-		(pin "3"
-		)
-		(pin "19"
-		)
-		(pin "8"
-		)
-		(pin "2"
-		)
-		(pin "9"
-		)
-		(pin "7"
-		)
-		(instances
-			(project ""
-				(path "/5f636c45-3c15-4731-8931-4625e0dab7e4/32de8c9e-be2b-4d78-9d5d-f4e694f2d2e7"
-					(reference "J9")
-					(unit 1)
-				)
