File: ftdi_level_shifters.kicad_sch (KiCad schematic)
At the start: 9 parts, among them U32 NTB0104_DHVQFN, U45 NTB0104_DHVQFN, U46 NTB0104_DHVQFN

Commit message: Update naming on schematics, fix OSM page size
Other:
- title: BMC Reference Carrier Board -> DC-SCM Carrier Card for OSM-L SoMs
Changed lines of the file:
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@@
 	(paper "A3")
 	(title_block
-		(title "BMC Reference Carrier Board")
-		(date "2025-10-13")
+		(title "DC-SCM Carrier Card for OSM-L SoMs")
+		(date "2025-10-14")
 		(rev "1.1.0")
 	)
